Commit message: ros_control error

File: andino_description/urdf/andino.urdf.xacro (robot description, xacro)
@@ -61,4 +61,4 @@
   </xacro:camera_sensor>
   <!-- ros2_control -->
-  <xacro:include filename="$(find ${package_name})/urdf/include/andino_control.urdf.xacro" />
+  <!-- <xacro:include filename="$(find ${package_name})/urdf/include/andino_control.urdf.xacro" /> -->
 </robot>

File: andino_gazebo/urdf/andino.gazebo.xacro (robot description, xacro)
@@ -16,4 +16,25 @@
   <xacro:friction reference="rear_caster_wheel_link" mu="0.05"/>
    <xacro:if value="$(arg use_gazebo_ros_control)">
+    <ros2_control name="GazeboSystem" type="system">
+    <hardware>
+      <plugin>gazebo_ros2_control/GazeboSystem</plugin>
+    </hardware>
+    <joint name="left_wheel_joint">
+      <command_interface name="velocity">
+        <param name="min">-5</param>
+        <param name="max">5</param>
+      </command_interface>
+      <state_interface name="velocity"/>
+      <state_interface name="position"/>
+    </joint>
+    <joint name="right_wheel_joint">
+      <command_interface name="velocity">
+        <param name="min">-5</param>
+        <param name="max">5</param>
+      </command_interface>
+      <state_interface name="velocity"/>
+      <state_interface name="position"/>
+    </joint>
+  </ros2_control>
     <gazebo>
       <plugin filename="libgazebo_ros2_control.so" name="gazebo_ros2_control">
@@ -27,5 +48,5 @@
   </xacro:if>
   <xacro:unless value="$(arg use_gazebo_ros_control)">
-	  <gazebo>
+	  <gazebo reference="robot">
     <plugin name="andino_joint_state" filename="libgazebo_ros_joint_state_publisher.so">
       <ros>
@@ -38,5 +59,5 @@
       <joint_name>left_wheel_joint</joint_name>
     </plugin>
-<plugin name='andino_diff_drive' filename='libgazebo_ros_diff_drive.so'>
+    <plugin name='andino_diff_drive' filename='libgazebo_ros_diff_drive.so'>
       <ros>
         <!-- <namespace>/andino</namespace> -->
@@ -61,7 +82,7 @@
 	  </gazebo>
   </xacro:unless>
-    <gazebo reference="base_link">
+    <gazebo reference="rplidar_laser_link">
       <sensor name="sensor_ray_front" type="ray">
-        <pose>0.05 0 0.06 0 0 -0</pose>
+        <!-- <pose>0.05 0 0.06 0 0 -0</pose> -->
         <ray>
           <scan>
@@ -98,7 +119,7 @@
     </gazebo>
   <!-- TODO: add the camera -->
-    <gazebo reference="base_link">
+    <gazebo reference="camera_link">
         <sensor name='camera' type='camera'>
-          <pose>0.085 0 0.01 0 -0 0</pose>
+          <!-- <pose>0.085 0 0.01 0 -0 0</pose> -->
           <camera>
             <horizontal_fov>1.047</horizontal_fov>
