Commit message: First commit
Signed-off-by: Gonzalo de Pedro <gonzalodepedro@ekumenlabs.com>

File: andino_description/urdf/include/common_macros.urdf.xacro (robot description, xacro)
@@ -62,5 +62,5 @@
       <child link="${prefix}_wheel"/>
       <origin xyz="${pos_x_joint} ${reflect* pos_y_joint} ${pos_z_joint}" rpy="0 0 0"/>
-      <dynamics damping="0.0" friction="4.5"/>
+      <dynamics damping="0.01" friction="0.0"/>
     </joint>
   </xacro:macro>

File: andino_gazebo/urdf/andino.gazebo.xacro (robot description, xacro)
@@ -6,12 +6,12 @@
       <mu1>${mu}</mu1>
       <mu2>${mu}</mu2>
-      <kp>1000000.0</kp>
+      <kp>1000000</kp>
       <kd>1.0</kd>
       <minDepth>0.0001</minDepth>
-      <maxVel>1.0</maxVel>
+      <maxVel>5.0</maxVel>
     </gazebo>
   </xacro:macro>
-  <xacro:friction reference="front_right_wheel" mu="100"/>
-  <xacro:friction reference="front_left_wheel" mu="100"/>
+  <xacro:friction reference="front_right_wheel" mu="0.7"/>
+  <xacro:friction reference="front_left_wheel" mu="0.7"/>
   <xacro:friction reference="rear_caster_wheel_link" mu="0.05"/>
    <xacro:if value="$(arg use_gazebo_ros_control)">
@@ -25,5 +25,4 @@
         <param name="max">5</param>
       </command_interface>
-      <state_interface name="velocity"/>
       <state_interface name="position"/>
     </joint>
@@ -33,5 +32,4 @@
         <param name="max">5</param>
       </command_interface>
-      <state_interface name="velocity"/>
       <state_interface name="position"/>
     </joint>
