Commit message: One Andino with diff_drive plugin

File: andino_description/urdf/include/andino_caster_macro.urdf.xacro (robot description, xacro)
@@ -28,8 +28,8 @@
           <geometry>
             <xacro:if value="${scale != '' }" >
-              <mesh filename="package://andino_description/meshes/${robot_name}/${wheel_props['base']['mesh']}" scale="${scale}"/>
+              <mesh filename="file://$(find andino_description)/meshes/${robot_name}/${wheel_props['base']['mesh']}" scale="${scale}"/>
             </xacro:if>
             <xacro:if value="${scale == '' }" >
-              <mesh filename="package://andino_description/meshes/${robot_name}/${wheel_props['base']['mesh']}" />
+              <mesh filename="file://$(find andino_description)/meshes/${robot_name}/${wheel_props['base']['mesh']}" />
             </xacro:if>
           </geometry>
@@ -78,8 +78,8 @@
           <geometry>
             <xacro:if value="${scale != '' }" >
-              <mesh filename="package://andino_description/meshes/${robot_name}/${wheel_props['hub']['mesh']}" scale="${scale}"/>
+              <mesh filename="file://$(find andino_description)/meshes/${robot_name}/${wheel_props['hub']['mesh']}" scale="${scale}"/>
             </xacro:if>
             <xacro:if value="${scale == '' }" >
-              <mesh filename="package://andino_description/meshes/${robot_name}/${wheel_props['hub']['mesh']}" />
+              <mesh filename="file://$(find andino_description)/meshes/${robot_name}/${wheel_props['hub']['mesh']}" />
             </xacro:if>
           </geometry>
@@ -127,8 +127,8 @@
           <geometry>
             <xacro:if value="${scale != '' }" >
-              <mesh filename="package://andino_description/meshes/${robot_name}/${wheel_props['wheel']['mesh']}" scale="${scale}"/>
+              <mesh filename="file://$(find andino_description)/meshes/${robot_name}/${wheel_props['wheel']['mesh']}" scale="${scale}"/>
             </xacro:if>
             <xacro:if value="${scale == '' }" >
-              <mesh filename="package://andino_description/meshes/${robot_name}/${wheel_props['wheel']['mesh']}" />
+              <mesh filename="file://$(find andino_description)/meshes/${robot_name}/${wheel_props['wheel']['mesh']}" />
             </xacro:if>
           </geometry>

File: andino_description/urdf/include/common_macros.urdf.xacro (robot description, xacro)
@@ -23,8 +23,8 @@
         <geometry>
           <xacro:if value="${wheel_props['scale'] == '' }" >
-            <mesh filename="package://andino_description/meshes/${robot_name}/${wheel_props['mesh']}" />
+            <mesh filename="file://$(find andino_description)/meshes/${robot_name}/${wheel_props['mesh']}" />
           </xacro:if>
           <xacro:if value="${wheel_props['scale'] == '' }" >
-            <mesh filename="package://andino_description/meshes/${robot_name}/${wheel_props['mesh']}" scale="${wheel_props['scale']}" />
+            <mesh filename="file://$(find andino_description)/meshes/${robot_name}/${wheel_props['mesh']}" scale="${wheel_props['scale']}" />
           </xacro:if>
         </geometry>
@@ -87,8 +87,8 @@
         <geometry>
           <xacro:if value="${motor_props['scale'] == '' }" >
-            <mesh filename="package://andino_description/meshes/${robot_name}/${motor_props['mesh']}" />
+            <mesh filename="file://$(find andino_description)/meshes/${robot_name}/${motor_props['mesh']}" />
           </xacro:if>
           <xacro:if value="${motor_props['scale'] != '' }" >
-            <mesh filename="package://andino_description/meshes/${robot_name}/${motor_props['mesh']}" scale="${motor_props['scale']}"/>
+            <mesh filename="file://$(find andino_description)/meshes/${robot_name}/${motor_props['mesh']}" scale="${motor_props['scale']}"/>
           </xacro:if>
         </geometry>
@@ -146,8 +146,8 @@
           <!-- The folder path get a folder_name global parameter -->
           <xacro:if value="${scale != '' }" >
-            <mesh filename="package://andino_description/meshes/${robot_name}/${mesh}" scale="${scale}"/>
+            <mesh filename="file://$(find andino_description)/meshes/${robot_name}/${mesh}" scale="${scale}"/>
           </xacro:if>
           <xacro:if value="${scale == '' }" >
-            <mesh filename="package://andino_description/meshes/${robot_name}/${mesh}" />
+            <mesh filename="file://$(find andino_description)/meshes/${robot_name}/${mesh}" />
           </xacro:if>
         </geometry>

File: andino_description/urdf/include/common_sensors.urdf.xacro (robot description, xacro)
@@ -9,5 +9,5 @@
       <origin xyz="0 0 0" rpy="0 0 ${pi}"/>
       <geometry>
-        <mesh filename="package://andino_description/meshes/sensors/${mesh}" />
+        <mesh filename="file://$(find andino_description)/meshes/sensors/${mesh}" />
       </geometry>
       <material name="dark_grey"/>
@@ -50,5 +50,5 @@
         <origin xyz="0 0 0" rpy="0 0 0"/>
         <geometry>
-          <mesh filename="package://${package_name}/meshes/sensors/${mesh}" />
+          <mesh filename="file://${package_name}/meshes/sensors/${mesh}" />
         </geometry>
         <material name="blue"/>

Commit message: from file to package in the xacro
Signed-off-by: olmerg <olmerg@gmail.com>

File: andino_description/urdf/include/andino_caster_macro.urdf.xacro (robot description, xacro)
@@ -28,8 +28,8 @@
           <geometry>
             <xacro:if value="${scale != '' }" >
-              <mesh filename="file://$(find andino_description)/meshes/${robot_name}/${wheel_props['base']['mesh']}" scale="${scale}"/>
+              <mesh filename="package://andino_description/meshes/${robot_name}/${wheel_props['base']['mesh']}" scale="${scale}"/>
             </xacro:if>
             <xacro:if value="${scale == '' }" >
-              <mesh filename="file://$(find andino_description)/meshes/${robot_name}/${wheel_props['base']['mesh']}" />
+              <mesh filename="package://andino_description/meshes/${robot_name}/${wheel_props['base']['mesh']}" />
             </xacro:if>
           </geometry>
@@ -78,8 +78,8 @@
           <geometry>
             <xacro:if value="${scale != '' }" >
-              <mesh filename="file://$(find andino_description)/meshes/${robot_name}/${wheel_props['hub']['mesh']}" scale="${scale}"/>
+              <mesh filename="package://andino_description/meshes/${robot_name}/${wheel_props['hub']['mesh']}" scale="${scale}"/>
             </xacro:if>
             <xacro:if value="${scale == '' }" >
-              <mesh filename="file://$(find andino_description)/meshes/${robot_name}/${wheel_props['hub']['mesh']}" />
+              <mesh filename="package://andino_description/meshes/${robot_name}/${wheel_props['hub']['mesh']}" />
             </xacro:if>
           </geometry>
@@ -127,8 +127,8 @@
           <geometry>
             <xacro:if value="${scale != '' }" >
-              <mesh filename="file://$(find andino_description)/meshes/${robot_name}/${wheel_props['wheel']['mesh']}" scale="${scale}"/>
+              <mesh filename="package://andino_description/meshes/${robot_name}/${wheel_props['wheel']['mesh']}" scale="${scale}"/>
             </xacro:if>
             <xacro:if value="${scale == '' }" >
-              <mesh filename="file://$(find andino_description)/meshes/${robot_name}/${wheel_props['wheel']['mesh']}" />
+              <mesh filename="package://andino_description/meshes/${robot_name}/${wheel_props['wheel']['mesh']}" />
             </xacro:if>
           </geometry>

File: andino_description/urdf/include/common_macros.urdf.xacro (robot description, xacro)
@@ -23,8 +23,8 @@
         <geometry>
           <xacro:if value="${wheel_props['scale'] == '' }" >
-            <mesh filename="file://$(find andino_description)/meshes/${robot_name}/${wheel_props['mesh']}" />
+            <mesh filename="package://andino_description/meshes/${robot_name}/${wheel_props['mesh']}" />
           </xacro:if>
           <xacro:if value="${wheel_props['scale'] == '' }" >
-            <mesh filename="file://$(find andino_description)/meshes/${robot_name}/${wheel_props['mesh']}" scale="${wheel_props['scale']}" />
+            <mesh filename="package://andino_description/meshes/${robot_name}/${wheel_props['mesh']}" scale="${wheel_props['scale']}" />
           </xacro:if>
         </geometry>
@@ -87,8 +87,8 @@
         <geometry>
           <xacro:if value="${motor_props['scale'] == '' }" >
-            <mesh filename="file://$(find andino_description)/meshes/${robot_name}/${motor_props['mesh']}" />
+            <mesh filename="package://andino_description/meshes/${robot_name}/${motor_props['mesh']}" />
           </xacro:if>
           <xacro:if value="${motor_props['scale'] != '' }" >
-            <mesh filename="file://$(find andino_description)/meshes/${robot_name}/${motor_props['mesh']}" scale="${motor_props['scale']}"/>
+            <mesh filename="package://andino_description/meshes/${robot_name}/${motor_props['mesh']}" scale="${motor_props['scale']}"/>
           </xacro:if>
         </geometry>
@@ -146,8 +146,8 @@
           <!-- The folder path get a folder_name global parameter -->
           <xacro:if value="${scale != '' }" >
-            <mesh filename="file://$(find andino_description)/meshes/${robot_name}/${mesh}" scale="${scale}"/>
+            <mesh filename="package://andino_description/meshes/${robot_name}/${mesh}" scale="${scale}"/>
           </xacro:if>
           <xacro:if value="${scale == '' }" >
-            <mesh filename="file://$(find andino_description)/meshes/${robot_name}/${mesh}" />
+            <mesh filename="package://andino_description/meshes/${robot_name}/${mesh}" />
           </xacro:if>
         </geometry>

File: andino_description/urdf/include/common_sensors.urdf.xacro (robot description, xacro)
@@ -9,5 +9,5 @@
       <origin xyz="0 0 0" rpy="0 0 ${pi}"/>
       <geometry>
-        <mesh filename="file://$(find andino_description)/meshes/sensors/${mesh}" />
+        <mesh filename="package://andino_description/meshes/sensors/${mesh}" />
       </geometry>
       <material name="dark_grey"/>
@@ -50,5 +50,5 @@
         <origin xyz="0 0 0" rpy="0 0 0"/>
         <geometry>
-          <mesh filename="file://${package_name}/meshes/sensors/${mesh}" />
+          <mesh filename="package://andino_description/meshes/sensors/${mesh}" />
         </geometry>
         <material name="blue"/>

File: andino_gazebo/urdf/andino.gazebo.xacro (robot description, xacro)
@@ -17,5 +17,6 @@
    <xacro:if value="$(arg use_gazebo_ros_control)">
     <gazebo>
-      <plugin name="gazebo_ros_control" filename="libgazebo_ros_control.so">
+      <plugin filename="libgazebo_ros2_control.so" name="gazebo_ros2_control">
+      <parameters>$(find andino_control)/config/andino_controllers.yaml</parameters>
           <!-- <robotNamespace>: The ROS namespace to be used for this instance of the plugin, defaults to robot name in URDF/SDF -->
           <!-- <controlPeriod>: The period of the controller update (in seconds), defaults to Gazebo's period -->
@@ -31,4 +32,5 @@
         <!-- <namespace>/andino</namespace> -->
         <remapping>~/out:=joint_states</remapping>
+        <remapping>/tf:=tf</remapping>
       </ros>
       <update_rate>10</update_rate>
@@ -40,4 +42,5 @@
         <!-- <namespace>/andino</namespace> -->
         <remapping>odom:=odom</remapping>
+        <remapping>/tf:=tf</remapping>
       </ros>
       <!-- wheels -->
@@ -95,3 +98,37 @@
     </gazebo>
   <!-- TODO: add the camera -->
+    <gazebo reference="base_link">
+        <sensor name='camera' type='camera'>
+          <pose>0.085 0 0.01 0 -0 0</pose>
+          <camera>
+            <horizontal_fov>1.047</horizontal_fov>
+            <image>
+              <width>640</width>
+              <height>480</height>
+            </image>
+            <clip>
+              <near>0.1</near>
+              <far>100</far>
+            </clip>
+          </camera>
+          <always_on>1</always_on>
+          <update_rate>30</update_rate>
+          <plugin name='camera_controller' filename='libgazebo_ros_camera.so'>
+            <alwaysOn>1</alwaysOn>
+            <cameraName>camera</cameraName>
+            <imageTopicName>image_raw</imageTopicName>
+            <cameraInfoTopicName>camera_info</cameraInfoTopicName>
+            <frameName>camera_link</frameName>
+            <hackBaseline>0.07</hackBaseline>
+            <distortionK1>0.0</distortionK1>
+            <distortionK2>0.0</distortionK2>
+            <distortionK3>0.0</distortionK3>
+            <distortionT1>0.0</distortionT1>
+            <distortionT2>0.0</distortionT2>
+            <!-- <ros>
+              <namespace>andino</namespace>
+            </ros> -->
+          </plugin>
+        </sensor>
+  </gazebo>
 </robot>

Commit message: Changed caster
Signed-off-by: Gonzalo de Pedro <gonzalodepedro@ekumenlabs.com>

File: andino_description/urdf/include/andino_caster_macro.urdf.xacro (robot description, xacro)
@@ -104,5 +104,5 @@
       </collision>
     </link>
-    <joint name="caster_rotation_joint" type="fixed">
+    <joint name="caster_rotation_joint" type="continuous">
       <origin xyz="${wheel_props['hub']['dx']} ${-wheel_props['hub']['dy'] * locationright} ${wheel_props['hub']['dz']}"
               rpy="0 0 0" />
@@ -153,5 +153,5 @@
       </collision>
     </link>
-    <joint name="caster_wheel_joint" type="fixed">
+    <joint name="caster_wheel_joint" type="continuous">
       <origin xyz="${wheel_props['wheel']['dx']} ${-wheel_props['wheel']['dy'] * locationright} ${wheel_props['wheel']['dz']}"
               rpy="0 0 0" />
